File: BassKatze/BassKatze.sch (KiCad schematic (older format))
At the start: 49 parts, among them J1 Conn_01x02_Female, Q1 IRF7404, Q2 BSS138, SW1 SW_Push, U1 ATmega328-AU, U2 MSGEQ7, U3 TP4056

Commit message: fixed charging circuit cuttoff not working, updated pcb to schematic
Parts:
- removed Charge_Powerup1: D, Diode_SMD:D_1206_3216Metric, symbol Device:D
Connections:
- wire segments 137 -> 135
Changed lines of the file:
@@
 	-1   0    0    1
 $EndComp
-$Comp
-L Device:D Charge_Powerup1
-U 1 1 5DB1380F
-P 1950 2300
-F 0 "Charge_Powerup1" H 1950 2084 50  0000 C CNN
-F 1 "D" H 1950 2175 50  0000 C CNN
-F 2 "Diode_SMD:D_1206_3216Metric" H 1950 2300 50  0001 C CNN
-F 3 "~" H 1950 2300 50  0001 C CNN
-	1    1950 2300
-	-1   0    0    1
-$EndComp
-Wire Wire Line
-	2100 2600 2100 2300
 Connection ~ 2100 2600
 Wire Wire Line
 	1650 2600 1800 2600
-Text GLabel 1800 2250 1    50   Input ~ 0
-5V_IN
-Wire Wire Line
-	1800 2250 1800 2300
 $Comp
 L Connector:Conn_01x02_Male BAT1

Commit message: force poweron, if isp is connected
Parts:
- added D18, D19: D, Diode_SMD:D_1206_3216Metric_Pad1.42x1.75mm_HandSolder, symbol Device:D
Connections:
- net labels added: 5V_Flash
- wire segments 135 -> 137
- no-connect marks 12 -> 11
Changed lines of the file:
@@
 	1    0    0    -1
 $EndComp
-Text GLabel 800  4300 3    50   Input ~ 0
+Text GLabel 800  4600 3    50   Input ~ 0
 PWR_HOLD
 Text GLabel 4800 3300 2    50   Input ~ 0
@@
 NoConn ~ 3550 1100
 NoConn ~ 1150 7050
-NoConn ~ 1200 1150
 Text GLabel 5650 1950 2    50   Input ~ 0
 PWR
@@
 Wire Wire Line
 	4750 2000 5200 2000
+$Comp
+L Device:D D18
+U 1 1 5DD2FE3A
+P 800 4450
+F 0 "D18" V 754 4529 50  0000 L CNN
+F 1 "D" V 845 4529 50  0000 L CNN
+F 2 "Diode_SMD:D_1206_3216Metric_Pad1.42x1.75mm_HandSolder" H 800 4450 50  0001 C CNN
+F 3 "~" H 800 4450 50  0001 C CNN
+	1    800  4450
+	0    1    1    0
+$EndComp
+$Comp
+L Device:D D19
+U 1 1 5DD309CE
+P 950 4300
+F 0 "D19" H 950 4516 50  0000 C CNN
+F 1 "D" H 950 4425 50  0000 C CNN
+F 2 "Diode_SMD:D_1206_3216Metric_Pad1.42x1.75mm_HandSolder" H 950 4300 50  0001 C CNN
+F 3 "~" H 950 4300 50  0001 C CNN
+	1    950  4300
+	1    0    0    -1
+$EndComp
+Connection ~ 800  4300
+Text GLabel 1150 4300 2    50   Input ~ 0
+5V_Flash
+Wire Wire Line
+	1100 4300 1150 4300
+Text GLabel 1150 1150 0    50   Input ~ 0
+5V_Flash
+Wire Wire Line
+	1150 1150 1200 1150
 $EndSCHEMATC

Commit message: add pretective resistor to data pin of arduino
Parts:
- added R14: 470Ohm, Resistor_SMD:R_1206_3216Metric_Pad1.42x1.75mm_HandSolder, symbol Device:R
Connections:
- wire segments 137 -> 138
Changed lines of the file:
@@
 Text GLabel 5600 2750 2    50   Input ~ 0
 EQ_Reset
-Text GLabel 4800 3000 2    50   Input ~ 0
+Text GLabel 5650 3000 2    50   Input ~ 0
 LED1
 Wire Wire Line
@@
 Wire Wire Line
 	1150 1150 1200 1150
+$Comp
+L Device:R R14
+U 1 1 5DD5D3A9
+P 4950 3000
+F 0 "R14" V 4743 3000 50  0000 C CNN
+F 1 "470Ohm" V 4834 3000 50  0000 C CNN
+F 2 "Resistor_SMD:R_1206_3216Metric_Pad1.42x1.75mm_HandSolder" V 4880 3000 50  0001 C CNN
+F 3 "~" H 4950 3000 50  0001 C CNN
+	1    4950 3000
+	0    1    1    0
+$EndComp
+Wire Wire Line
+	5650 3000 5100 3000
 $EndSCHEMATC

Commit message: Added R16, added modes to sketch
Parts:
- added R15: 10k, Resistor_SMD:R_1206_3216Metric_Pad1.42x1.75mm_HandSolder, symbol Device:R
Changed lines of the file:
@@
 Wire Wire Line
 	5650 3000 5100 3000
+$Comp
+L Device:R R15
+U 1 1 5DEED760
+P 1800 2450
+F 0 "R15" H 1870 2496 50  0000 L CNN
+F 1 "10k" H 1870 2405 50  0000 L CNN
+F 2 "Resistor_SMD:R_1206_3216Metric_Pad1.42x1.75mm_HandSolder" V 1730 2450 50  0001 C CNN
+F 3 "~" H 1800 2450 50  0001 C CNN
+	1    1800 2450
+	1    0    0    -1
+$EndComp
+Connection ~ 1800 2600
+Text GLabel 1800 2300 1    50   Input ~ 0
+GND
 $EndSCHEMATC

Commit message: use TP5400 to remove issues with isp voltage
Parts:
- removed D1, D18, D19: D, Diode_SMD:D_1206_3216Metric_Pad1.42x1.75mm_HandSolder, symbol Device:D
- removed Q1: IRF7404, Package_SO:SOIC-8_3.9x4.9mm_P1.27mm, symbol Transistor_FET:IRF7404
- removed Q2: BSS138, Package_TO_SOT_SMD:SOT-23, symbol Transistor_FET:BSS138
- removed R10, R8: 5KOhm, Resistor_SMD:R_1206_3216Metric_Pad1.42x1.75mm_HandSolder, symbol Device:R
- removed R11, R12, R13: 10KOhm, Resistor_SMD:R_1206_3216Metric_Pad1.42x1.75mm_HandSolder, symbol Device:R
- removed R7, R9: 1KOhm, Resistor_SMD:R_1206_3216Metric_Pad1.42x1.75mm_HandSolder, symbol Device:R
- removed RProg1: 1.2kOhm, Resistor_SMD:R_1206_3216Metric_Pad1.42x1.75mm_HandSolder, symbol Device:R
- removed U3: TP4056, tp4056:TP4056_SOP-8-PP, symbol tp4056:TP4056
- added C10, C8: 22uF, Capacitor_SMD:C_0805_2012Metric, symbol Device:C
- added C7: 0.1uF, Capacitor_SMD:C_0805_2012Metric, symbol Device:C
- added C9: 47uF, Capacitor_SMD:C_0805_2012Metric, symbol Device:C
- added D1: 3A 20V, Diode_SMD:D_1206_3216Metric, symbol Device:D_Schottky
- added L1: 10uH, Inductor_SMD:L_1210_3225Metric, symbol Device:L
- added U3: TP5400, tp4056:TP4056_SOP-8-PP, symbol tp4056:TP5400
- added U4: TS5A3166DBVR, Package_TO_SOT_SMD:SOT-23-5, symbol Analog_Switch:TS5A3166DBVR
- C1: footprint Resistor_SMD:R_1206_3216Metric_Pad1.42x1.75mm_HandSolder -> Capacitor_SMD:C_0805_2012Metric
- C2: value 10uF -> 0.1uF; footprint Resistor_SMD:R_1206_3216Metric_Pad1.42x1.75mm_HandSolder -> Capacitor_SMD:C_0805_2012Metric
- R1: value 0.4Ohm -> 0.2Ohm; footprint Resistor_SMD:R_1206_3216Metric_Pad1.42x1.75mm_HandSolder -> Resistor_SMD:R_0805_2012Metric
- R4: value 10KOhm -> 1.2KOhm; footprint Resistor_SMD:R_1206_3216Metric_Pad1.42x1.75mm_HandSolder -> Resistor_SMD:R_0805_2012Metric
Connections:
- net labels added: BAT+_Switched
- net labels removed: PWR_HOLD
- wire segments 138 -> 128
- no-connect marks 11 -> 9

Commit message: update of the layout
Signed-off-by: Kai Boernert <kai-boernert@visiongamestudios.de>
Parts:
- C3, C4, C5, C6, R14, R15, R2, R3, R5, R6: footprint Resistor_SMD:R_1206_3216Metric_Pad1.42x1.75mm_HandSolder -> Resistor_SMD:R_0805_2012Metric_Pad1.15x1.40mm_HandSolder
- R1: footprint Resistor_SMD:R_0805_2012Metric -> Resistor_SMD:R_1206_3216Metric_Pad1.42x1.75mm_HandSolder
Connections:
- wire segments 128 -> 127
- no-connect marks 9 -> 7
Changed lines of the file:
@@
 F 0 "C3" V 7558 2100 50  0000 C CNN
 F 1 "0.1uF" V 7649 2100 50  0000 C CNN
-F 2 "Resistor_SMD:R_1206_3216Metric_Pad1.42x1.75mm_HandSolder" V 7740 2100 50  0000 C CNN
+F 2 "Resistor_SMD:R_0805_2012Metric_Pad1.15x1.40mm_HandSolder" V 7740 2100 50  0000 C CNN
 F 3 "~" H 7900 2100 50  0001 C CNN
 	1    7900 2100
@@
 F 0 "R2" V 6843 2500 50  0000 C CNN
 F 1 "26KOhm" V 6934 2500 50  0000 C CNN
-F 2 "Resistor_SMD:R_1206_3216Metric_Pad1.42x1.75mm_HandSolder" V 6980 2500 50  0001 C CNN
+F 2 "Resistor_SMD:R_0805_2012Metric_Pad1.15x1.40mm_HandSolder" V 6980 2500 50  0001 C CNN
 F 3 "~" H 7050 2500 50  0001 C CNN
 	1    7050 2500
@@
 F 0 "C6" H 9265 2696 50  0000 L CNN
 F 1 "0.1uF" H 9265 2605 50  0000 L CNN
-F 2 "Resistor_SMD:R_1206_3216Metric_Pad1.42x1.75mm_HandSolder" H 9188 2500 50  0001 C CNN
+F 2 "Resistor_SMD:R_0805_2012Metric_Pad1.15x1.40mm_HandSolder" H 9188 2500 50  0001 C CNN
 F 3 "~" H 9150 2650 50  0001 C CNN
 	1    9150 2650
@@
 F 0 "C4" H 8165 2596 50  0000 L CNN
 F 1 "33pF" H 8165 2505 50  0000 L CNN
-F 2 "Resistor_SMD:R_1206_3216Metric_Pad1.42x1.75mm_HandSolder" H 8088 2400 50  0001 C CNN
+F 2 "Resistor_SMD:R_0805_2012Metric_Pad1.15x1.40mm_HandSolder" H 8088 2400 50  0001 C CNN
 F 3 "~" H 8050 2550 50  0001 C CNN
 	1    8050 2550
@@
 F 0 "R3" V 7643 2400 50  0000 C CNN
 F 1 "200KOhm" V 7734 2400 50  0000 C CNN
-F 2 "Resistor_SMD:R_1206_3216Metric_Pad1.42x1.75mm_HandSolder" V 7780 2400 50  0001 C CNN
+F 2 "Resistor_SMD:R_0805_2012Metric_Pad1.15x1.40mm_HandSolder" V 7780 2400 50  0001 C CNN
 F 3 "~" H 7850 2400 50  0001 C CNN
 	1    7850 2400
@@
 F 0 "C5" V 8248 1500 50  0000 C CNN
 F 1 "0.1uF" V 8339 1500 50  0000 C CNN
-F 2 "Resistor_SMD:R_1206_3216Metric_Pad1.42x1.75mm_HandSolder" H 8538 1350 50  0001 C CNN
+F 2 "Resistor_SMD:R_0805_2012Metric_Pad1.15x1.40mm_HandSolder" H 8538 1350 50  0001 C CNN
 F 3 "~" H 8500 1500 50  0001 C CNN
 	1    8500 1500
@@
 F 0 "R5" H 5120 2746 50  0000 L CNN
 F 1 "10KOhm" H 5120 2655 50  0000 L CNN
-F 2 "Resistor_SMD:R_1206_3216Metric_Pad1.42x1.75mm_HandSolder" V 4980 2700 50  0001 C CNN
+F 2 "Resistor_SMD:R_0805_2012Metric_Pad1.15x1.40mm_HandSolder" V 4980 2700 50  0000 C CNN
 F 3 "~" H 5050 2700 50  0001 C CNN
 	1    5050 2700
@@
 	8050 2700 8050 2750
 Connection ~ 8050 2700
-NoConn ~ 4750 1800
-NoConn ~ 4750 1700
 NoConn ~ 4750 1300
 NoConn ~ 4750 1200
@@
 F 0 "R6" V 6693 2350 50  0000 C CNN
 F 1 "147KOhm" V 6784 2350 50  0000 C CNN
-F 2 "Resistor_SMD:R_1206_3216Metric_Pad1.42x1.75mm_HandSolder" V 6830 2350 50  0001 C CNN
+F 2 "Resistor_SMD:R_0805_2012Metric_Pad1.15x1.40mm_HandSolder" V 6830 2350 50  0001 C CNN
 F 3 "~" H 6900 2350 50  0001 C CNN
 	1    6900 2350
@@
 	4250 800  4150 800
 Connection ~ 4150 800
-Wire Wire Line
-	5650 1950 5600 1950
 Wire Wire Line
 	4750 2600 5200 2600
@@
 F 0 "R1" V 1893 6150 50  0000 C CNN
 F 1 "0.2Ohm" V 1984 6150 50  0000 C CNN
-F 2 "Resistor_SMD:R_0805_2012Metric" V 2030 6150 50  0001 C CNN
+F 2 "Resistor_SMD:R_1206_3216Metric_Pad1.42x1.75mm_HandSolder" V 2030 6150 50  0001 C CNN
 F 3 "~" H 2100 6150 50  0001 C CNN
 	1    2100 6150
@@
 F 0 "R15" H 2770 3346 50  0000 L CNN
 F 1 "10k" H 2770 3255 50  0000 L CNN
-F 2 "Resistor_SMD:R_1206_3216Metric_Pad1.42x1.75mm_HandSolder" V 2630 3300 50  0001 C CNN
+F 2 "Resistor_SMD:R_0805_2012Metric_Pad1.15x1.40mm_HandSolder" V 2630 3300 50  0001 C CNN
 F 3 "~" H 2700 3300 50  0001 C CNN
 	1    2700 3300
@@
 F 0 "R14" V 4743 3000 50  0000 C CNN
 F 1 "470Ohm" V 4834 3000 50  0000 C CNN
-F 2 "Resistor_SMD:R_1206_3216Metric_Pad1.42x1.75mm_HandSolder" V 4880 3000 50  0001 C CNN
+F 2 "Resistor_SMD:R_0805_2012Metric_Pad1.15x1.40mm_HandSolder" V 4880 3000 50  0001 C CNN
 F 3 "~" H 4950 3000 50  0001 C CNN
 	1    4950 3000

Commit message: 0.7 low voltage cutoff mosfet
Parts:
- added 10K1: R, Resistor_SMD:R_0805_2012Metric, symbol Device:R
- added Q1: Q_PMOS_GDS, Package_TO_SOT_SMD:SOT-23, symbol Device:Q_PMOS_GDS
Connections:
- wire segments 127 -> 128
Changed lines of the file:
@@
 Wire Wire Line
 	8650 2600 8650 2700
-Text GLabel 4900 5850 2    50   Input ~ 0
+Text GLabel 5300 6300 2    50   Input ~ 0
 PWR
 Text GLabel 4800 3200 2    50   Input ~ 0
@@
 Wire Wire Line
 	3150 6900 3150 6800
-Text GLabel 4900 6150 2    50   Input ~ 0
+Text GLabel 4350 6150 3    50   Input ~ 0
 GND
 $Comp
@@
 	1    0    0    -1
 $EndComp
-Wire Wire Line
-	4900 5850 4550 5850
 Connection ~ 4550 5850
 Wire Wire Line
@@
 	3650 5850 3650 6150
 Connection ~ 4100 5850
-Wire Wire Line
-	4900 6150 4550 6150
-Connection ~ 4550 6150
 Wire Wire Line
 	4550 6150 4100 6150
@@
 Wire Wire Line
 	4800 2300 4750 2300
+$Comp
+L Device:Q_PMOS_GDS Q1
+U 1 1 5E3890D3
+P 5300 6100
+F 0 "Q1" H 5505 6054 50  0000 L CNN
+F 1 "Q_PMOS_GDS" H 5505 6145 50  0000 L CNN
+F 2 "Package_TO_SOT_SMD:SOT-23" H 5500 6200 50  0001 C CNN
+F 3 "~" H 5300 6100 50  0001 C CNN
+	1    5300 6100
+	-1   0    0    1
+$EndComp
+Wire Wire Line
+	4550 5850 5200 5850
+Text GLabel 5800 6100 2    50   Input ~ 0
+BAT+
+Wire Wire Line
+	5200 5850 5200 5900
+Wire Wire Line
+	5300 6300 5200 6300
+$Comp
+L Device:R 10K1
+U 1 1 5E3A2A18
+P 5650 6100
+F 0 "10K1" V 5443 6100 50  0000 C CNN
+F 1 "R" V 5534 6100 50  0000 C CNN
+F 2 "Resistor_SMD:R_0805_2012Metric" V 5580 6100 50  0001 C CNN
+F 3 "~" H 5650 6100 50  0001 C CNN
+	1    5650 6100
+	0    1    1    0
+$EndComp
 $EndSCHEMATC
