File: BassKatze/BassKatze.sch (KiCad schematic (older format))
At the start: 52 parts, among them J1 Conn_01x02_Female, Q1 IRF7404, Q2 BSS138, SW1 SW_Push, U1 ATmega328-AU, U2 MSGEQ7, U3 TP4056

Commit message: use voltage converters to prevent isp burnout
Parts:
- removed R11, R12, R13, R4: 10KOhm, Resistor_SMD:R_1206_3216Metric_Pad1.42x1.75mm_HandSolder, symbol Device:R
- added Q3, Q4, Q5, Q6: BSS138, Package_TO_SOT_SMD:SOT-23, symbol Transistor_FET:BSS138
- added RN1, RN3: R_Pack04, Resistor_SMD:R_Array_Convex_4x0603, symbol Device:R_Pack04
- added RN2: R_Pack0410K, Resistor_SMD:R_Array_Convex_4x0603, symbol Device:R_Pack04
- C1, C2, C3, C4, C5, C6: footprint Resistor_SMD:R_1206_3216Metric_Pad1.42x1.75mm_HandSolder -> Capacitor_SMD:C_0805_2012Metric
- D1, D18, D19: footprint Diode_SMD:D_1206_3216Metric_Pad1.42x1.75mm_HandSolder -> Diode_SMD:D_SOD-323
- J1: footprint Connector_PinHeader_2.54mm:PinHeader_1x02_P2.54mm_Vertical -> Resistor_SMD:R_0603_1608Metric
- MIC1: footprint Connector_PinHeader_2.54mm:PinHeader_1x05_P2.54mm_Vertical -> Connector_PinHeader_2.54mm:PinHeader_1x06_P2.54mm_Vertical; symbol Connector:Conn_01x05_Male -> Connector:Conn_01x06_Male
- R1: value 0.4Ohm -> 0.2Ohm
- R10, R14, R15, R2, R3, R6, R7, R8, R9, RProg1: footprint Resistor_SMD:R_1206_3216Metric_Pad1.42x1.75mm_HandSolder -> Resistor_SMD:R_0603_1608Metric
- R5: footprint Resistor_SMD:R_1206_3216Metric_Pad1.42x1.75mm_HandSolder -> Resistor_SMD:R_0805_2012Metric
Connections:
- net labels added: Free1, MISO_5V, MOSI_5V, Reset_5V, SCK_5V
- wire segments 138 -> 181
- no-connect marks 11 -> 10

Commit message: tracing of 0.8 finished
Parts:
- R10, R14, R15, R2, R3, R6, R7, R8, R9, RProg1: footprint Resistor_SMD:R_0603_1608Metric -> Resistor_SMD:R_0805_2012Metric
- renumbered BAT1 to +Bat-1, Charge1 to +Charge-1, ISP1 to ISP_5v1

Commit message: basskatze 0.9 -> removed redundant reset pullup
Parts:
- removed R5: 10KOhm, Resistor_SMD:R_0805_2012Metric, symbol Device:R
Connections:
- wire segments 181 -> 173
Changed lines of the file:
@@
 Text GLabel 5700 1250 2    50   Input ~ 0
 RAW_Spectrum
-Text GLabel 5650 2250 2    50   Input ~ 0
+Text GLabel 5700 2600 2    50   Input ~ 0
 Reset
 $Comp
@@
 Wire Wire Line
 	4750 1600 4850 1600
-Text GLabel 5600 2650 2    50   Input ~ 0
+Text GLabel 5700 2400 2    50   Input ~ 0
 EQ_Band
-Text GLabel 5600 2750 2    50   Input ~ 0
+Text GLabel 5700 2500 2    50   Input ~ 0
 EQ_Reset
 Text GLabel 5650 3000 2    50   Input ~ 0
@@
 	1050 6350 1350 6350
 Connection ~ 1350 6350
-$Comp
-L Device:R R5
-U 1 1 5DB0845E
-P 5600 2100
-F 0 "R5" H 5670 2146 50  0000 L CNN
-F 1 "10KOhm" H 5670 2055 50  0000 L CNN
-F 2 "Resistor_SMD:R_0805_2012Metric" V 5530 2100 50  0001 C CNN
-F 3 "~" H 5600 2100 50  0001 C CNN
-	1    5600 2100
-	-1   0    0    1
-$EndComp
 Text GLabel 4800 3400 2    50   Input ~ 0
 CHRG
@@
 NoConn ~ 3550 1100
 NoConn ~ 9450 4500
-Text GLabel 5650 1950 2    50   Input ~ 0
-PWR
 Wire Wire Line
 	8200 1000 9850 1000
@@
 Wire Wire Line
 	4750 2200 4800 2200
-Wire Wire Line
-	5600 2650 5600 2400
-Wire Wire Line
-	5600 2400 4750 2400
-Wire Wire Line
-	4750 2500 5500 2500
-Wire Wire Line
-	5500 2500 5500 2750
-Wire Wire Line
-	5500 2750 5600 2750
 $Comp
 L Connector:Conn_01x02_Female J1
@@
 	4250 800  4150 800
 Connection ~ 4150 800
-Wire Wire Line
-	5650 2250 5600 2250
-Wire Wire Line
-	5650 1950 5600 1950
-Wire Wire Line
-	5600 2250 5600 2350
-Wire Wire Line
-	5600 2350 5350 2350
-Wire Wire Line
-	5350 2350 5350 2600
-Wire Wire Line
-	4750 2600 5350 2600
-Connection ~ 5600 2250
 $Comp
 L Device:R R8
@@
 	1    0    0    -1
 $EndComp
+Wire Wire Line
+	4750 2400 5700 2400
+Wire Wire Line
+	4750 2500 5700 2500
+Wire Wire Line
+	4750 2600 5700 2600
 $EndSCHEMATC

Commit message: basskatze 1.0 (fixed diode footprint, better manually solderable resistor arrays)
Parts:
- D1, D18, D19: footprint Diode_SMD:D_SOD-323 -> Diode_SMD:D_0805_2012Metric_Pad1.15x1.40mm_HandSolder
- RN1, RN2: footprint Resistor_SMD:R_Array_Convex_4x0603 -> Resistor_SMD:R_Array_Convex_4x1206
Changed lines of the file:
@@
 F 0 "D1" H 2150 1184 50  0000 C CNN
 F 1 "D" H 2150 1275 50  0000 C CNN
-F 2 "Diode_SMD:D_SOD-323" H 2150 1400 50  0001 C CNN
+F 2 "Diode_SMD:D_0805_2012Metric_Pad1.15x1.40mm_HandSolder" H 2150 1400 50  0001 C CNN
 F 3 "~" H 2150 1400 50  0001 C CNN
 	1    2150 1400
@@
 F 0 "D18" V 1304 2579 50  0000 L CNN
 F 1 "D" V 1395 2579 50  0000 L CNN
-F 2 "Diode_SMD:D_SOD-323" H 1350 2500 50  0001 C CNN
+F 2 "Diode_SMD:D_0805_2012Metric_Pad1.15x1.40mm_HandSolder" H 1350 2500 50  0001 C CNN
 F 3 "~" H 1350 2500 50  0001 C CNN
 	1    1350 2500
@@
 F 0 "D19" H 1500 2866 50  0000 C CNN
 F 1 "D" H 1500 2775 50  0000 C CNN
-F 2 "Diode_SMD:D_SOD-323" H 1500 2650 50  0001 C CNN
+F 2 "Diode_SMD:D_0805_2012Metric_Pad1.15x1.40mm_HandSolder" H 1500 2650 50  0001 C CNN
 F 3 "~" H 1500 2650 50  0001 C CNN
 	1    1500 2650
@@
 F 0 "RN1" H 2388 4196 50  0000 L CNN
 F 1 "R_Pack04" H 2388 4105 50  0000 L CNN
-F 2 "Resistor_SMD:R_Array_Convex_4x0603" V 2475 4150 50  0001 C CNN
+F 2 "Resistor_SMD:R_Array_Convex_4x1206" V 2475 4150 50  0001 C CNN
 F 3 "~" H 2200 4150 50  0001 C CNN
 	1    2200 4150
@@
 Wire Wire Line
 	5150 5300 5150 4500
-$Comp
-L Device:R_Pack04 RN3
-U 1 1 5E5E4B48
-P 3150 4150
-F 0 "RN3" H 3338 4196 50  0000 L CNN
-F 1 "R_Pack04" H 3338 4105 50  0000 L CNN
-F 2 "Resistor_SMD:R_Array_Convex_4x0603" V 3425 4150 50  0001 C CNN
-F 3 "~" H 3150 4150 50  0001 C CNN
-	1    3150 4150
-	1    0    0    -1
-$EndComp
 Text GLabel 2950 3950 1    50   Input ~ 0
 PWR
-Wire Wire Line
-	2950 3950 3050 3950
-Connection ~ 3050 3950
-Wire Wire Line
-	3050 3950 3150 3950
-Connection ~ 3150 3950
-Wire Wire Line
-	3150 3950 3250 3950
 Wire Wire Line
 	1600 4350 2000 4350
@@
 	4700 4650 4700 5300
 Connection ~ 4700 5300
-$Comp
-L Device:R_Pack04 RN2
-U 1 1 5E680DA3
-P 2700 2700
-F 0 "RN2" H 2888 2746 50  0000 L CNN
-F 1 "R_Pack0410K" H 2888 2655 50  0000 L CNN
-F 2 "Resistor_SMD:R_Array_Convex_4x0603" V 2975 2700 50  0001 C CNN
-F 3 "~" H 2700 2700 50  0001 C CNN
-	1    2700 2700
-	1    0    0    -1
-$EndComp
 Wire Wire Line
 	2700 3100 2700 2900
@@
 Wire Wire Line
 	4750 2600 5700 2600
+$Comp
+L Device:R_Pack04 RN2
+U 1 1 5E680DA3
+P 2700 2700
+F 0 "RN2" H 2888 2746 50  0000 L CNN
+F 1 "R_Pack0410K" H 2888 2655 50  0000 L CNN
+F 2 "Resistor_SMD:R_Array_Convex_4x1206" V 2975 2700 50  0001 C CNN
+F 3 "~" H 2700 2700 50  0001 C CNN
+	1    2700 2700
+	1    0    0    -1
+$EndComp
+Wire Wire Line
+	2950 3950 3050 3950
+Connection ~ 3050 3950
+Wire Wire Line
+	3150 3950 3250 3950
+Wire Wire Line
+	3050 3950 3150 3950
+Connection ~ 3150 3950
+$Comp
+L Device:R_Pack04 RN3
+U 1 1 5E5E4B48
+P 3150 4150
+F 0 "RN3" H 3338 4196 50  0000 L CNN
+F 1 "R_Pack04" H 3338 4105 50  0000 L CNN
+F 2 "Resistor_SMD:R_Array_Convex_4x0603" V 3425 4150 50  0001 C CNN
+F 3 "~" H 3150 4150 50  0001 C CNN
+	1    3150 4150
+	1    0    0    -1
+$EndComp
 $EndSCHEMATC
